File: hw/giris/giris.kicad_sch (KiCad schematic)
At the start: 0 parts

Commit message: Draw the 32-key giris schematic
Scales the six-key osu pad up to one half of the split keyboard. The
sheet was an empty A4 stub; it is now an A2 root with 32 hierarchical
instances of a new key.kicad_sch.

Per key, unchanged from the pad as corrected: TMR2615x sensor on +3.3VA,
30 pF at the source into 5.1 k and 3.3 nF at the mux, a Kailh
CPG151101S11-16 hotswap socket across the analog node, an SK6812MINI-E
in the chain, and 2 x 100 nF.

Top level: AT32F405RBT7-7, four TMUX1574RSVR muxes taking 32 sensors down
to ADC1_IN0-IN15 on one shared SEL line, three USB-C ports, the LM66100 /
AP22653 power path and XC6206 + TPS7A4700 rails carried over from the
pad, 12 MHz crystal, two buttons, three fiducials. The XC6206 symbol here
already has the corrected 1=VSS 2=VOUT 3=VIN pinout. No layout yet — the
.kicad_pcb is still a stub.

Project file gains the netclasses the pad uses plus one per mux group
(ADC_A..ADC_D), drops default clearance to 0.16 mm, and tightens ERC:
pin_to_pin to error, and the dangling-global-label and pin-map checks
switched on.
Parts:
- added C1, C2, C3, C4, C5, C6: CL21A226MAQNNNE, Capacitor_SMD:C_0805_2012Metric, symbol Basic_Capacitors_Resistors__C:CL21A226MAQNNNE
- added C11, C131, C19, C23, C25, C26, C27, C28, C29, C30, C65, C8, C98: CL05B104KB54PNC, Capacitor_SMD:C_0402_1005Metric, symbol Basic_Capacitors_Resistors__C:CL05B104KB54PNC
- added C12, C13, C20, C21, C7: CL21A106KAYNNNE, Capacitor_SMD:C_0805_2012Metric, symbol Basic_Capacitors_Resistors__C:CL21A106KAYNNNE
- added C14, C22: CL05A105KA5NQNC, Capacitor_SMD:C_0402_1005Metric, symbol Basic_Capacitors_Resistors__C:CL05A105KA5NQNC
- added C15, C16, C17, C18, C31, C32: 0402CG300J500NT, Capacitor_SMD:C_0402_1005Metric, symbol Basic_Capacitors_Resistors__C:0402CG300J500NT
- added C24: CL10A475KO8NNNC, Capacitor_SMD:C_0603_1608Metric, symbol Basic_Capacitors_Resistors__C:CL10A475KO8NNNC
- added C9: CL21A476MQYNNNE, Capacitor_SMD:C_0805_2012Metric, symbol Basic_Capacitors_Resistors__C:CL21A476MQYNNNE
- added D1: 1N4148WS_T4, Diode_SMD:D_SOD-323_HandSoldering, symbol Diode__C:1N4148WS_T4
- added FID1, FID2, FID3: Fiducial, Fiducial:Fiducial_1mm_Mask2mm, symbol Mechanical:Fiducial
- added H1, H2, H3: MountingHole_Pad, MountingHole:MountingHole_2.2mm_M2_Pad_Via, symbol Mechanical:MountingHole_Pad
- added J1, J2, J3: TYPE-C-31-M-12, Connector_USB__C:USB-C_SMD-TYPE-C-31-M-12_1, symbol Connector_USB__C:TYPE-C-31-M-12
- added J4: XY-SH1_0-4A61, Connector_SH1.0__C:CONN-SMD_4P-P1.00_XYECONN_XY-SH1.0-4A61, symbol Connector_SH1.0__C:XY-SH1_0-4A61
- added J6: Conn_01x23, Connector_PinHeader_2.54mm:PinHeader_1x23_P2.54mm_Vertical, symbol Connector_Generic:Conn_01x23
- added J8: Conn_01x04, Connector_PinHeader_2.54mm:PinHeader_1x04_P2.54mm_Vertical, symbol Connector_Generic:Conn_01x04
- added J9: (no value), Connector:Tag-Connect_TC2030-IDC-NL_2x03_P1.27mm_Vertical, symbol Connector:TC2030
- added L1: GZ1608D601TF, Inductor_SMD:L_0603_1608Metric, symbol Inductor__C:GZ1608D601TF
- added LED1, LED2: KT-0603W, LED__C:LED0603-R-RD_WHITE, symbol LED__C:KT-0603W
- added R1, R10, R2, R28, R5, R6: 0402WGF1002TCE, Resistor_SMD:R_0402_1005Metric, symbol Basic_Capacitors_Resistors__C:0402WGF1002TCE
- added R11: 0402WGF2202TCE, Resistor_SMD:R_0402_1005Metric, symbol Basic_Capacitors_Resistors__C:0402WGF2202TCE
- added R12, R13, R15, R17, R18, R19, R20, R22: 0402WGF5101TCE, Resistor_SMD:R_0402_1005Metric, symbol Basic_Capacitors_Resistors__C:0402WGF5101TCE
- added R14, R16, R21, R27, R3, R7: 0402WGF1200TCE, Resistor_SMD:R_0402_1005Metric, symbol Basic_Capacitors_Resistors__C:0402WGF1200TCE
- added R23, R24: 0402WGF3300TCE, Resistor_SMD:R_0402_1005Metric, symbol Basic_Capacitors_Resistors__C:0402WGF3300TCE
- added R25: 0402WGF1202TCE, Resistor_SMD:R_0402_1005Metric, symbol Basic_Capacitors_Resistors__C:0402WGF1202TCE
- added R26: 0402WGF3301TCE, Resistor_SMD:R_0402_1005Metric, symbol Basic_Capacitors_Resistors__C:0402WGF3301TCE
- added SW1, SW2: SKSGPAE010, Switch__C:SW-SMD_SKSGAAE010, symbol Switch__C:SKSGPAE010
- added TP1, TP10, TP11, TP12, TP13, TP14, TP15, TP16, TP2, TP3, TP4, TP5, TP7, TP8, TP9: TestPoint, TestPoint:TestPoint_Pad_D1.0mm, symbol Connector:TestPoint
- added U1, U5, U9: SRV05-4A, Diode__C:SOT-23-6, symbol Diode__C:SRV05-4
- added U10: AT32F405RBT7-7, MCU_Artery__C:LQFP-64_L7.0-W7.0-P0.40-LS9.0-BL, symbol MCU_Artery__C:AT32F405RBT7-7
- added U11, U31, U48, U65: TMUX1574RSVR, MUX__C:UQFN-16_L2.6-W1.8-P0.40-BL, symbol MUX__C:TMUX1574RSVR
- added U12: SK6812MINI-E, LED__C:LED-SMD_4P-L3.2-W2.8-LS5.9_SK6812MINI-E, symbol LED__C:SK6812MINI-E_C5149201
- added U2, U7: LM66100DCK, Package_TO_SOT_SMD:SOT-363_SC-70-6, symbol Power_Management:LM66100DCK
- added U25, U26: PESD5V0R1BSFYL, Diode__C:SOD-962_L0.6-W0.3-BI, symbol Diode__C:PESD5V0R1BSFYL
- added U3: AP22653W6-7, Power_Switch__C:SOT-23-6_L2.9-W1.6-P0.95-LS2.8-BR, symbol Power_Switch__C:AP22653W6-7
- added U4: TPS7A4700, Regulator_Linear__C:VQFN-20_L5.0-W5.0-P0.65-TL-EP, symbol Regulator_Linear__C:TPS7A4700
- added U8: XC6206P332MR, Regulator_Linear__C:SOT-23-3_L2.9-W1.6-P1.90-LS2.8-BR, symbol Regulator_Linear__C:XC6206P332MR
- added X1: X322512MSB4SI, Oscillator__C:X322512MSB4SI, symbol Oscillator__C:X322512MSB4SI
Connections:
- new net: R27.1, U12.2 (DIN)
- new net: R27.2, U10.62 (PB9)
- new net: C22.1, C23.2, L1.1, U10.13 (VDDA)
- new net: LED1.2 (K), R23.1
- new net: J1.A6 (DP1), J1.B6 (DP2), R7.1, TP1.1
- new net: J4.4, R16.2
- new net: J1.A5 (CC1), R13.2
- new net: J1.A7 (DN1), J1.B7 (DN2), R3.1, TP2.1
- new net: J1.B5 (CC2), R12.2
- new net: J3.A5 (CC1), R20.2
- new net: J2.B5 (CC2), R17.2
- new net: R11.2, U3.5 (ILIM)
- new net: R14.1, R15.2, R22.2
- new net: C29.2, D1.1 (K), U12.3 (VDD)
- new net: J2.A5 (CC1), R18.2
- new net: J3.B5 (CC2), R19.2
- new net: C14.2, U4.14 (NR)
- new net: LED2.2 (K), R24.1
- new net: J4.3, R21.2
- new net +3.3V: C21.1, C24.1, C25.2, C26.2, C27.2, J4.2, J6.4 (Pin_4), J8.2 (Pin_2), LED2.1 (A), R1.2, R14.2, R2.2, R28.2, R5.2, R6.2, SW1.1, SW1.3, TP12.1, U1.5 (VP), U10.1 (VDD), U10.36 (VDD), U10.64 (VDD), U8.2 (Vout), U9.5 (VP)
- new net +3.3VA: C131.2, C28.2, C65.2, C9.2, C98.2, L1.2, LED1.1 (A), TP3.1, U11.14 (VDD), U31.14 (VDD), U4.1 (OUT), U4.20 (OUT), U4.3 (SENSE/FB), U48.14 (VDD), U65.14 (VDD)
- new net +5V: C1.2, C13.2, C19.2, C2.2, C20.2, C3.2, C4.2, C5.2, C6.2, D1.2 (A), J6.3 (Pin_3), TP11.1, U2.3 (~{CE}), U2.6 (VOUT), U4.13 (EN), U4.15 (IN), U4.16 (IN), U5.5 (VP), U7.3 (~{CE}), U7.6 (VOUT), U8.3 (Vin)
- new net ADC1_IN0: TP13.1, U10.14 (PA0), U11.10 (D4)
- new net ADC1_IN1: TP14.1, U10.15 (PA1), U11.7 (D3)
- new net ADC1_IN10: U10.8 (PC0), U48.5 (D2)
- new net ADC1_IN11: U10.9 (PC1), U48.2 (D1)
- new net ADC1_IN12: U10.10 (PC2), U65.10 (D4)
- new net ADC1_IN13: U10.11 (PC3), U65.7 (D3)
- new net ADC1_IN14: U10.24 (PC4), U65.5 (D2)
- new net ADC1_IN15: U10.25 (PC5), U65.2 (D1)
- new net ADC1_IN2: TP15.1, U10.16 (PA2), U11.5 (D2)
- new net ADC1_IN3: TP16.1, U10.17 (PA3), U11.2 (D1)
- new net ADC1_IN4: U10.20 (PA4), U31.10 (D4)
- new net ADC1_IN5: U10.21 (PA5), U31.7 (D3)
- new net ADC1_IN6: U10.22 (PA6), U31.5 (D2)
- new net ADC1_IN7: U10.23 (PA7), U31.2 (D1)
- new net ADC1_IN8: U10.26 (PB0), U48.10 (D4)
- new net ADC1_IN9: U10.27 (PB1), U48.7 (D3)
- new net AP_FAULT: R6.1, TP7.1, U10.29 (PB10), U3.4 (FAULT#)
- new net BOOT: R26.2, SW1.2, SW1.4, U10.60 (PF11/BOOT0)
- new net DIN: U12.4 (DOUT)
- new net GND: C1.1, C11.1, C12.2, C13.1, C131.1, C14.1, C15.1, C16.1, C17.1, C18.1, C19.1, C2.1, C20.1, C21.2, C22.2, C23.1, C24.2, C25.1, C26.1, C27.1, C28.1, C29.1, C3.1, C30.1, C31.2, C32.1, C4.1, C5.1, C6.1, C65.1, C7.2, C8.1, C9.1, C98.1, H1.1, H2.1, H3.1, J1.1 (EH), J1.2 (EH), J1.3 (EH), J1.4 (EH), J1.A1B12 (GND), J1.B1A12 (GND), J2.1 (EH), J2.2 (EH), J2.3 (EH), J2.4 (EH), J2.A1B12 (GND), J2.B1A12 (GND), J3.1 (EH), J3.2 (EH), J3.3 (EH), J3.4 (EH), J3.A1B12 (GND), J3.B1A12 (GND), J4.1, J4.5, J4.6, J6.1 (Pin_1), J6.16 (Pin_16), J6.2 (Pin_2), J8.1 (Pin_1), J9.1, R10.1, R11.1, R12.1, R13.1, R17.1, R18.1, R19.1, R20.1, R23.2, R24.2, R25.1, R26.1, SW1.5, SW1.6, SW2.2, SW2.4, SW2.5, SW2.6, TP9.1, U1.2 (VN), U10.12 (VSSA), U10.31 (VSS), U10.63 (VSS), U11.13 (EN#), U11.6 (GND), U12.1 (GND), U2.2 (GND), U25.1, U26.1, U3.2 (GND), U31.13 (EN#), U31.6 (GND), U4.11 (0P2V), U4.12 (0P1V), U4.17 (NC), U4.18 (NC), U4.19 (NC), U4.2 (NC), U4.21 (TP), U4.7 (GND), U4.8 (1P6V), U48.13 (EN#), U48.6 (GND), U5.2 (VN), U65.13 (EN#), U65.6 (GND), U7.2 (GND), U7.5 (ST), U8.1 (GND), U9.2 (VN), X1.2 (GND), X1.4 (GND)
- new net I2C1_SCL: R16.1, R22.1, U10.19 (PF5), U9.3 (IO2), U9.4 (IO3)
- new net I2C1_SDA: R15.1, R21.1, U10.18 (PF4), U9.1 (IO1), U9.6 (IO4)
- new net I2C2_SCL: J6.11 (Pin_11), U10.47 (PF6)
- new net I2C2_SDA: J6.10 (Pin_10), U10.48 (PF7)
- new net I2C3_SCL: J8.4 (Pin_4), U10.32 (PB13)
- new net I2C3_SDA: J8.3 (Pin_3), U10.56 (PB4)
- new net IO1: J6.17 (Pin_17), U10.54 (PD2)
- new net IO2: J6.18 (Pin_18), U10.57 (PB5)
- new net IO3: J6.19 (Pin_19), U10.58 (PB6)
- new net IO4: J6.20 (Pin_20), U10.59 (PB7)
- new net IO5: J6.21 (Pin_21), U10.61 (PB8)
- new net IO6: J6.22 (Pin_22), U10.3 (PC14)
- new net IO7: J6.23 (Pin_23), U10.4 (PC15)
- new net LM_ST: R5.1, TP5.1, U10.30 (PB12), U2.5 (ST)
- new net OTGFS1_D+: C15.2, J2.A6 (DP1), J2.B6 (DP2), U10.45 (PA12), U5.1 (IO1), U5.6 (IO4)
- new net OTGFS1_D-: C16.2, J2.A7 (DN1), J2.B7 (DN2), U10.44 (PA11), U5.3 (IO2), U5.4 (IO3)
- new net OTGHS1_D+: C17.2, J3.A6 (DP1), J3.B6 (DP2), U10.35 (OTGHS1_D+), U25.2
- new net OTGHS1_D-: C18.2, J3.A7 (DN1), J3.B7 (DN2), U10.34 (OTGHS1_D-), U26.2
- new net OTGHS1_R: R25.2, U10.33 (OTGHS1_R)
- new net PW_PSTRH: R10.2, TP8.1, U10.2 (PC13), U3.3 (EN/EN#)
- new net RCC_OSC_IN: C31.1, U10.5 (PF0), X1.1 (OSC1)
- new net RCC_OSC_OUT: C32.2, U10.6 (PF1), X1.3 (OSC2)
- new net RESET: C30.2, R28.1, SW2.1, SW2.3, U10.7 (NRST)
- new net SPI3_CS: J6.12 (Pin_12), U10.50 (PA15)
- new net SPI3_MISO: J6.14 (Pin_14), U10.52 (PC11)
- new net SPI3_MOSI: J6.15 (Pin_15), U10.53 (PC12)
- new net SPI3_SCK: J6.13 (Pin_13), U10.51 (PC10)
- new net SWO: J9.6, U10.55 (PB3)
- new net SYS_SWCLK: J9.4, U10.49 (PA14)
- new net SYS_SWDIO: J9.2, U10.46 (PA13)
- new net TMUXA_S1A: U11.16 (S1A)
- new net TMUXA_S1B: U11.1 (S1B)
- new net TMUXA_S2A: U11.3 (S2A)
- new net TMUXA_S2B: U11.4 (S2B)
- new net TMUXA_S3A: U11.9 (S3A)
- new net TMUXA_S3B: U11.8 (S3B)
- new net TMUXA_S4A: U11.12 (S4A)
- new net TMUXA_S4B: U11.11 (S4B)
- new net TMUXB_S1A: U31.16 (S1A)
- new net TMUXB_S1B: U31.1 (S1B)
- new net TMUXB_S2A: U31.3 (S2A)
- new net TMUXB_S2B: U31.4 (S2B)
- new net TMUXB_S3A: U31.9 (S3A)
- new net TMUXB_S3B: U31.8 (S3B)
- new net TMUXB_S4A: U31.12 (S4A)
- new net TMUXB_S4B: U31.11 (S4B)
- new net TMUXC_S1A: U48.16 (S1A)
- new net TMUXC_S1B: U48.1 (S1B)
- new net TMUXC_S2A: U48.3 (S2A)
- new net TMUXC_S2B: U48.4 (S2B)
- new net TMUXC_S3A: U48.9 (S3A)
- new net TMUXC_S3B: U48.8 (S3B)
- new net TMUXC_S4A: U48.12 (S4A)
- new net TMUXC_S4B: U48.11 (S4B)
- new net TMUXD_S1A: U65.16 (S1A)
- new net TMUXD_S1B: U65.1 (S1B)
- new net TMUXD_S2A: U65.3 (S2A)
- new net TMUXD_S2B: U65.4 (S2B)
- new net TMUXD_S3A: U65.9 (S3A)
- new net TMUXD_S3B: U65.8 (S3B)
- new net TMUXD_S4A: U65.12 (S4A)
- new net TMUXD_S4B: U65.11 (S4B)
- new net TMUX_SEL: U10.28 (PB2), U11.15 (SEL), U31.15 (SEL), U48.15 (SEL), U65.15 (SEL)
- new net UART7_RX: R2.1, R3.2, U1.1 (IO1), U1.6 (IO4), U10.37 (PC6)
- new net UART7_TX: R1.1, R7.2, U1.3 (IO2), U1.4 (IO3), U10.38 (PC7)
- new net UART8_RX: J6.6 (Pin_6), U10.40 (PC9)
- new net UART8_TX: J6.5 (Pin_5), U10.39 (PC8)
- new net USART1_CK: J6.9 (Pin_9), U10.41 (PA8)
- new net USART1_RX: J6.7 (Pin_7), J9.5, U10.43 (PA10)
- new net USART1_TX: J6.8 (Pin_8), J9.3, U10.42 (PA9)
- new net VBUS_B: C11.2, C12.1, J1.A4B9 (VBUS), J1.B4A9 (VBUS), TP4.1, U2.1 (VIN), U3.6 (OUT)
- new net VBUS_HOST: C7.1, C8.2, J3.A4B9 (VBUS), J3.B4A9 (VBUS), TP10.1, U3.1 (IN), U7.1 (VIN)
- no-connect marks 0 -> 14
Other:
- added sheet Key (key.kicad_sch)
- added sheet Key1 (key.kicad_sch)
- added sheet Key10 (key.kicad_sch)
- added sheet Key11 (key.kicad_sch)
- added sheet Key12 (key.kicad_sch)
- added sheet Key13 (key.kicad_sch)
- added sheet Key14 (key.kicad_sch)
- added sheet Key15 (key.kicad_sch)
- added sheet Key16 (key.kicad_sch)
- added sheet Key17 (key.kicad_sch)
- added sheet Key18 (key.kicad_sch)
- added sheet Key19 (key.kicad_sch)
- added sheet Key2 (key.kicad_sch)
- added sheet Key20 (key.kicad_sch)
- added sheet Key21 (key.kicad_sch)
- added sheet Key22 (key.kicad_sch)
- added sheet Key23 (key.kicad_sch)
- added sheet Key24 (key.kicad_sch)
- added sheet Key25 (key.kicad_sch)
- added sheet Key26 (key.kicad_sch)
- added sheet Key27 (key.kicad_sch)
- added sheet Key28 (key.kicad_sch)
- added sheet Key29 (key.kicad_sch)
- added sheet Key3 (key.kicad_sch)
- added sheet Key30 (key.kicad_sch)
- added sheet Key31 (key.kicad_sch)
- added sheet Key4 (key.kicad_sch)
- added sheet Key5 (key.kicad_sch)
- added sheet Key6 (key.kicad_sch)
- added sheet Key7 (key.kicad_sch)
- added sheet Key8 (key.kicad_sch)
- added sheet Key9 (key.kicad_sch)
- note added: "APWR LED"
- note added: "BOOT SW"
- note added: "DPWR LED"
- note added: "HSE Oscillator"
- note added: "QWIIC Pullup jumper"
- note added: "RESET SW"
- note added: "TagConnect Debug Header TC2030-NL"
